File: dragon-pcb.kicad_pcb (KiCad board)
At the start: 2 copper layers, 64.4 x 98.6 mm, 12 parts, among them M1 Motor_DC, Q1 NPN, SW1 SW_Push

Commit message: Add files via upload
Parts:
- added G***: LOGO, LOGO, B.Cu at (94.5, 114.5)
- added R4: R, Resistor_THT:R_Axial_DIN0207_L6.3mm_D2.5mm_P7.62mm_Horizontal, B.Cu at (115.0, 129.9)
- added R5: R, Resistor_THT:R_Axial_DIN0207_L6.3mm_D2.5mm_P7.62mm_Horizontal, B.Cu at (115.0, 134.0)
Connections:
- D3 pad 2: Net-(D1-A) -> Net-(D3-A)
- D4 pad 2: Net-(D1-A) -> Net-(D3-A)
- D5 pad 2: Net-(D1-A) -> Net-(D5-A)
Routing:
- net Net-(D5-A): track 0.00 -> 66.0 mm, vias 0 -> 1
- net Net-(D1-A): track 134.4 -> 79.5 mm
- net Net-(D3-A): track 0.00 -> 33.7 mm, vias 0 -> 1
- net Net-(BT1-+): track 174.0 -> 189.7 mm

Commit message: Add files via upload
Parts:
- removed G***: LOGO, LOGO
- moved R1 2.50 mm to (93.7, 79.5)
Routing:
- net Net-(Q1-B): track 86.8 -> 81.5 mm
- net Net-(BT1--): track 117.1 -> 114.6 mm
