File: dragon-pcb.kicad_sch (KiCad schematic)
At the start: 12 parts, among them M1 Motor_DC, Q1 NPN, SW1 SW_Push

Commit message: Add files via upload
Parts:
- added R4, R5: R, Resistor_THT:R_Axial_DIN0207_L6.3mm_D2.5mm_P7.62mm_Horizontal, symbol Device:R
Connections:
- net at D1.2 (A), D2.2 (A), R2.2: no longer D3.2 (A), D4.2 (A), D5.2 (A)
- net at BT1.1 (+), R2.1, R3.1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: now also R4.1, R5.1
- new net: D5.2 (A), R5.2
- new net: D3.2 (A), D4.2 (A), R4.2
Other:
- moved on the sheet: D5, R2

Commit message: Add files via upload
Changed lines of the file:
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@@
 	(wire
 		(pts
-			(xy 128.27 25.4) (xy 128.27 49.53)
+			(xy 128.27 25.4) (xy 128.27 46.99)
 		)
 		(stroke
@@
 	(wire
 		(pts
-			(xy 128.27 57.15) (xy 128.27 72.39)
+			(xy 128.27 54.61) (xy 128.27 72.39)
 		)
 		(stroke
@@
 	(symbol
 		(lib_id "Device:Battery_Cell")
-		(at 128.27 54.61 0)
+		(at 128.27 52.07 0)
 		(unit 1)
 		(exclude_from_sim no)
@@
 		(fields_autoplaced yes)
 		(property "Reference" "BT1"
+			(at 132.08 48.9584 0)
+			(effects
+				(font
+					(size 1.27 1.27)
+				)
+				(justify left)
+			)
+		)
+		(property "Value" "Battery_Cell"
 			(at 132.08 51.4984 0)
 			(effects
@@
 			)
 		)
-		(property "Value" "Battery_Cell"
-			(at 132.08 54.0384 0)
-			(effects
-				(font
-					(size 1.27 1.27)
-				)
-				(justify left)
-			)
-		)
 		(property "Footprint" "Battery:BatteryHolder_Keystone_3034_1x20mm"
-			(at 128.27 53.086 90)
-			(effects
-				(font
-					(size 1.27 1.27)
-				)
-				(hide yes)
-			)
-		)
-		(property "Datasheet" "~"
-			(at 128.27 53.086 90)
+			(at 128.27 50.546 90)
+			(effects
+				(font
+					(size 1.27 1.27)
+				)
+				(hide yes)
+			)
+		)
+		(property "Datasheet" "~"
+			(at 128.27 50.546 90)
 			(effects
 				(font
@@
 		)
 		(property "Description" "Single-cell battery"
-			(at 128.27 54.61 0)
-			(effects
-				(font
+			(at 128.27 52.07 0)
+			(effects
+				(font
